File: mini_mouse.brd (EAGLE design)
At the start: 92 x 92 mm, 32 parts, among them IC1 PIC18F4550_TQFP, IC3 LP2950CDT-5.0, IC4 L293D

Commit message: Final Designe
Parts:
- C3, C4: device rcl:E5-6 -> rcl:E2-4
- moved RS1 0.61 mm to (15.4, 73.4)
Routing:
- net BAT: track 100.0 -> 101.5 mm
- net +5V: track 415.9 -> 416.8 mm
Other:
- board text added: "UAQ"
Changed lines of the file:
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@@
 <setting verticaltext="up"/>
 </settings>
-<grid distance="3" unitdist="mil" unit="mm" style="lines" multiple="1" display="no" altdistance="5" altunitdist="mil" altunit="mm"/>
+<grid distance="3" unitdist="mil" unit="mil" style="lines" multiple="1" display="no" altdistance="5" altunitdist="mil" altunit="mil"/>
 <layers>
 <layer number="1" name="Top" color="4" fill="1" visible="yes" active="yes"/>
@@
 <wire x1="7" y1="62" x2="7" y2="30" width="0.254" layer="20"/>
 <wire x1="7" y1="30" x2="0" y2="30" width="0.254" layer="20"/>
+<text x="13.5636" y="13.6398" size="5.08" layer="16" font="vector" rot="MR0">UAQ</text>
 </plain>
 <attributes>
@@
 <attribute name="VALUE" x="34.163" y="68.682003125" size="1.27" layer="27" ratio="10" rot="R270"/>
 </element>
-<element name="RS1" library="rcl" library_urn="urn:adsk.eagle:library:334" package="R0805" package3d_urn="urn:adsk.eagle:package:23553/2" value="" x="15.3928" y="73.9646" rot="MR270">
-<attribute name="NAME" x="14.7578" y="74.5996" size="1.27" layer="26" rot="MR270"/>
-<attribute name="SPICEPREFIX" value="R" x="75.0828" y="23.1646" size="1.778" layer="28" rot="MR270" display="off"/>
-<attribute name="VALUE" x="17.2978" y="74.5996" size="1.27" layer="28" rot="MR270"/>
+<element name="RS1" library="rcl" library_urn="urn:adsk.eagle:library:334" package="R0805" package3d_urn="urn:adsk.eagle:package:23553/2" value="" x="15.3928" y="73.355" rot="MR270">
+<attribute name="NAME" x="14.7578" y="73.99" size="1.27" layer="26" rot="MR270"/>
+<attribute name="SPICEPREFIX" value="R" x="75.0828" y="22.555" size="1.778" layer="28" rot="MR270" display="off"/>
+<attribute name="VALUE" x="17.2978" y="73.99" size="1.27" layer="28" rot="MR270"/>
 </element>
 <element name="RS2" library="rcl" library_urn="urn:adsk.eagle:library:334" package="R0805" package3d_urn="urn:adsk.eagle:package:23553/2" value="" x="15.3922" y="77.8764" rot="MR90">
@@
 <attribute name="VALUE" x="38.304" y="19.854" size="1.27" layer="27" ratio="10"/>
 </element>
-<element name="C3" library="rcl" library_urn="urn:adsk.eagle:library:334" package="E5-6" package3d_urn="urn:adsk.eagle:package:23368/1" value="" x="81.61" y="22.631" rot="R180">
+<element name="C3" library="rcl" library_urn="urn:adsk.eagle:library:334" package="E2-4" package3d_urn="urn:adsk.eagle:package:23347/1" value="" x="81.61" y="22.631" rot="R180">
 <attribute name="NAME" x="78.562" y="20.853" size="1.27" layer="25" ratio="10" rot="R180"/>
 <attribute name="SPICEPREFIX" value="C" x="81.61" y="22.631" size="1.778" layer="27" rot="R180" display="off"/>
 <attribute name="VALUE" x="78.562" y="25.552" size="1.27" layer="27" ratio="10" rot="R180"/>
 </element>
-<element name="C4" library="rcl" library_urn="urn:adsk.eagle:library:334" package="E5-6" package3d_urn="urn:adsk.eagle:package:23368/1" value="" x="77.013" y="27.915" rot="R180">
+<element name="C4" library="rcl" library_urn="urn:adsk.eagle:library:334" package="E2-4" package3d_urn="urn:adsk.eagle:package:23347/1" value="" x="77.013" y="27.915" rot="R180">
 <attribute name="NAME" x="73.965" y="26.137" size="1.27" layer="25" ratio="10" rot="R180"/>
 <attribute name="SPICEPREFIX" value="C" x="77.013" y="27.915" size="1.778" layer="27" rot="R180" display="off"/>
@@
 <wire x1="27.051" y1="2.8194" x2="78.0288" y2="2.8194" width="0.6096" layer="16"/>
 <wire x1="15.3924" y1="14.478" x2="27.051" y2="2.8194" width="0.508" layer="16"/>
-<wire x1="79.553" y1="27.915" x2="85.5472" y2="27.9146" width="0.6096" layer="16"/>
+<wire x1="78.029" y1="27.915" x2="85.5472" y2="27.9146" width="0.6096" layer="16"/>
 <wire x1="85.5472" y1="27.9146" x2="89.8398" y2="23.622" width="0.6096" layer="16"/>
 <wire x1="89.8398" y1="23.622" x2="89.8398" y2="11.3538" width="0.6096" layer="16"/>
 <wire x1="89.8398" y1="11.3538" x2="87.1728" y2="8.6868" width="0.6096" layer="16"/>
-<wire x1="79.553" y1="27.915" x2="75.5142" y2="23.876" width="0.6096" layer="16"/>
 <wire x1="75.5142" y1="23.876" x2="75.5142" y2="18.3074" width="0.6096" layer="16"/>
 <contactref element="COMUNICACION" pad="1"/>
@@
 <wire x1="33.54" y1="79.5" x2="33.54" y2="75" width="0.508" layer="16"/>
 <wire x1="33.54" y1="70.5" x2="33.54" y2="75" width="0.508" layer="16"/>
-<wire x1="33.54" y1="59.1192" x2="33.54" y2="59.436" width="0.508" layer="16"/>
-<wire x1="33.54" y1="59.436" x2="33.54" y2="70.5" width="0.508" layer="16"/>
+<wire x1="33.54" y1="58.46" x2="33.54" y2="70.5" width="0.508" layer="16"/>
 <wire x1="33.54" y1="84" x2="33.54" y2="86.2464" width="0.508" layer="16"/>
 <wire x1="33.54" y1="86.2464" x2="33.0708" y2="86.7156" width="0.508" layer="16"/>
@@
 <wire x1="1.397" y1="76.734" x2="1.397" y2="72.136" width="0.508" layer="16"/>
 <wire x1="41.89878125" y1="50.10121875" x2="33.54" y2="58.46" width="0.508" layer="16"/>
-<wire x1="33.54" y1="58.46" x2="33.54" y2="59.1192" width="0.508" layer="16"/>
+<wire x1="78.029" y1="27.915" x2="78.029" y2="26.3908" width="0.6096" layer="16"/>
+<wire x1="78.029" y1="26.3908" x2="75.5142" y2="23.876" width="0.6096" layer="16"/>
 </signal>
 <signal name="PGD">
@@
 <contactref element="JP1" pad="1"/>
 <contactref element="JP1" pad="3"/>
-<polygon width="0.508" layer="16" isolate="0.254">
+<polygon width="0.508" layer="16" isolate="0.2">
 <vertex x="0.2286" y="-0.381"/>
 <vertex x="92.583" y="-0.381"/>
@@
 <wire x1="11.6586" y1="81.6102" x2="17.2974" y2="81.6102" width="0.508" layer="1"/>
 <via x="17.2974" y="81.6102" extent="1-16" drill="0.6" diameter="1.3" shape="octagon"/>
-<wire x1="45.6788" y1="27.1272" x2="44.527" y2="25.9754" width="0.508" layer="16"/>
-<wire x1="44.527" y1="24.299" x2="44.527" y2="25.9754" width="0.508" layer="16"/>
-<wire x1="58.9788" y1="27.1272" x2="45.6788" y2="27.1272" width="0.508" layer="16"/>
+<wire x1="45.4502" y1="27.1272" x2="44.7556" y2="26.4326" width="0.508" layer="16"/>
+<wire x1="44.7556" y1="26.4326" x2="44.7556" y2="24.5276" width="0.508" layer="16"/>
+<wire x1="44.527" y1="24.299" x2="44.7556" y2="24.5276" width="0.508" layer="16"/>
+<wire x1="58.9788" y1="27.1272" x2="45.4502" y2="27.1272" width="0.508" layer="16"/>
 <wire x1="58.9788" y1="27.1272" x2="58.9788" y2="26.5938" width="0.508" layer="16"/>
 <wire x1="58.9788" y1="26.5938" x2="60.198" y2="25.3746" width="0.508" layer="16"/>
@@
 <contactref element="RS1" pad="1"/>
 <contactref element="IC1" pad="25"/>
-<wire x1="15.3928" y1="74.9146" x2="14.4642" y2="74.8146" width="0.508" layer="16"/>
-<wire x1="14.4642" y1="74.8146" x2="13.1064" y2="73.4568" width="0.508" layer="16"/>
+<wire x1="13.1064" y1="73.4568" x2="13.781028125" y2="74.131428125" width="0.508" layer="16"/>
 <wire x1="13.1064" y1="73.4568" x2="13.1064" y2="66.8274" width="0.508" layer="16"/>
 <via x="30.7086" y="63.0174" extent="1-16" drill="0.6" diameter="1.3" shape="octagon"/>
@@
 <wire x1="17.2212" y1="65.4558" x2="14.478" y2="65.4558" width="0.508" layer="16"/>
 <wire x1="14.478" y1="65.4558" x2="13.1064" y2="66.8274" width="0.508" layer="16"/>
+<wire x1="13.781028125" y1="74.131428125" x2="15.219228125" y2="74.131428125" width="0.508" layer="16"/>
+<wire x1="15.219228125" y1="74.131428125" x2="15.3928" y2="74.305" width="0.508" layer="16"/>
 </signal>
 <signal name="PA_2">
@@
 <wire x1="87.4014" y1="11.9634" x2="87.4014" y2="21.5646" width="0.6096" layer="16"/>
 <wire x1="87.4014" y1="21.5646" x2="86.3346" y2="22.6314" width="0.6096" layer="16"/>
-<wire x1="86.3346" y1="22.6314" x2="84.15" y2="22.631" width="0.6096" layer="16"/>
+<wire x1="86.3346" y1="22.6314" x2="82.626" y2="22.631" width="0.6096" layer="16"/>
 <wire x1="86.106" y1="10.668" x2="87.4014" y2="11.9634" width="0.6096" layer="16"/>
 <wire x1="82.4484" y1="10.668" x2="77.0382" y2="5.2578" width="0.6096" layer="16"/>
